File: circuits/dac-pcb/dac-pcb.kicad_pcb (KiCad board)
At the start: 2 copper layers, 46.7 x 18.8 mm, 50 parts, among them J1 Conn_01x18

Commit message: Added images kicad
Routing:
- added copper zone on B.Cu, net GND
- added copper zone on F.Cu, net GND
